File: RJ45-CAN-Distributor.kicad_pcb (KiCad board)
At the start: 2 copper layers, 66 x 115 mm, 18 parts, among them J1 RJ45_Amphenol_54602-x08_Horiz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

Commit message: Route, associate and generate bom and drawings.
Parts:
- J1: value RJ45_Amphenol_54602-x08_Horizontal -> RJ45
- J10, J2, J3, J4, J5, J6, J7, J8, J9: renamed from REF**; value RJ45_Amphenol_54602-x08_Horizontal -> RJ45
- R1: renamed from REF**; value R_Axial_DIN0411_L9.9mm_D3.6mm_P15.24mm_Horizontal -> 120
- moved G1 1.00 mm to (155.3, 117.2)
- moved J1 0.75 mm to (136.2, 55.7)
- moved J2 0.75 mm to (136.2, 74.4)
- moved J3 0.75 mm to (136.2, 93.2)
- moved J4 0.75 mm to (136.2, 113.2)
- moved J5 0.75 mm to (136.2, 133.2)
- renumbered REF** to G1, REF** to G2, REF** to H1, REF** to H2, REF** to H3, REF** to H4
Connections:
- J1 pad 1: (no net) -> CAN_H
- J1 pad 2: (no net) -> CAN_L
- J1 pad 3: (no net) -> CAN_GND
- J1 pad 4: (no net) -> Reserved1
- J1 pad 5: (no net) -> Reserved2
- J1 pad 6: (no net) -> SHIELD
- J1 pad 7: (no net) -> CAN_GND
- J1 pad 8: (no net) -> CAN_V+
- J10 pad 1: (no net) -> CAN_H
- J10 pad 2: (no net) -> CAN_L
- J10 pad 3: (no net) -> CAN_GND
- J10 pad 4: (no net) -> Reserved1
- J10 pad 5: (no net) -> Reserved2
- J10 pad 6: (no net) -> SHIELD
- J10 pad 7: (no net) -> CAN_GND
- J10 pad 8: (no net) -> CAN_V+
- J2 pad 1: (no net) -> CAN_H
- J2 pad 2: (no net) -> CAN_L
- J2 pad 3: (no net) -> CAN_GND
- J2 pad 4: (no net) -> Reserved1
- J2 pad 5: (no net) -> Reserved2
- J2 pad 6: (no net) -> SHIELD
- J2 pad 7: (no net) -> CAN_GND
- J2 pad 8: (no net) -> CAN_V+
- J3 pad 1: (no net) -> CAN_H
- J3 pad 2: (no net) -> CAN_L
- J3 pad 3: (no net) -> CAN_GND
- J3 pad 4: (no net) -> Reserved1
- J3 pad 5: (no net) -> Reserved2
- J3 pad 6: (no net) -> SHIELD
- J3 pad 7: (no net) -> CAN_GND
- J3 pad 8: (no net) -> CAN_V+
- J4 pad 1: (no net) -> CAN_H
- J4 pad 2: (no net) -> CAN_L
- J4 pad 3: (no net) -> CAN_GND
- J4 pad 4: (no net) -> Reserved1
- J4 pad 5: (no net) -> Reserved2
- J4 pad 6: (no net) -> SHIELD
- J4 pad 7: (no net) -> CAN_GND
- J4 pad 8: (no net) -> CAN_V+
- J5 pad 1: (no net) -> CAN_H
- J5 pad 2: (no net) -> CAN_L
- J5 pad 3: (no net) -> CAN_GND
- J5 pad 4: (no net) -> Reserved1
- J5 pad 5: (no net) -> Reserved2
- J5 pad 6: (no net) -> SHIELD
- J5 pad 7: (no net) -> CAN_GND
- J5 pad 8: (no net) -> CAN_V+
- J6 pad 1: (no net) -> CAN_H
- J6 pad 2: (no net) -> CAN_L
- J6 pad 3: (no net) -> CAN_GND
- J6 pad 4: (no net) -> Reserved1
- J6 pad 5: (no net) -> Reserved2
- J6 pad 6: (no net) -> SHIELD
- J6 pad 7: (no net) -> CAN_GND
- J6 pad 8: (no net) -> CAN_V+
- J7 pad 1: (no net) -> CAN_H
- J7 pad 2: (no net) -> CAN_L
- J7 pad 3: (no net) -> CAN_GND
- J7 pad 4: (no net) -> Reserved1
- J7 pad 5: (no net) -> Reserved2
- J7 pad 6: (no net) -> SHIELD
- J7 pad 7: (no net) -> CAN_GND
- J7 pad 8: (no net) -> CAN_V+
- J8 pad 1: (no net) -> CAN_H
- J8 pad 2: (no net) -> CAN_L
- J8 pad 3: (no net) -> CAN_GND
- J8 pad 4: (no net) -> Reserved1
- J8 pad 5: (no net) -> Reserved2
- J8 pad 6: (no net) -> SHIELD
- J8 pad 7: (no net) -> CAN_GND
- J8 pad 8: (no net) -> CAN_V+
- J9 pad 1: (no net) -> CAN_H
- J9 pad 2: (no net) -> CAN_L
- J9 pad 3: (no net) -> CAN_GND
- J9 pad 4: (no net) -> Reserved1
- J9 pad 5: (no net) -> Reserved2
- J9 pad 6: (no net) -> SHIELD
- J9 pad 7: (no net) -> CAN_GND
- J9 pad 8: (no net) -> CAN_V+
- R1 pad 1: (no net) -> CAN_L
- R1 pad 2: (no net) -> CAN_H
Routing:
- net CAN_GND: track 0.00 -> 314.7 mm, vias 0 -> 4
- net CAN_H: track 0.00 -> 307.7 mm, vias 0 -> 5
- net SHIELD: track 0.00 -> 276.9 mm, vias 0 -> 3
- net Reserved2: track 0.00 -> 266.0 mm, vias 0 -> 2
- net CAN_V+: track 0.00 -> 243.0 mm, vias 0 -> 5
- net Reserved1: track 0.00 -> 231.4 mm, vias 0 -> 4
- net CAN_L: track 0.00 -> 208.8 mm, vias 0 -> 4
Other:
- board text added: "*Optional external supply"
